File: mykeyboard/matrix.sch (KiCad schematic (older format))
At the start: 0 parts

Commit message: complete matrix
Parts:
- added D1, D10, D11, D12, D13, D14, D15, D16, D17, D18, D19, D2, D20, D21, D22, D23, D24, D25, D26, D27, D28, D29, D3, D30, D31, D32, D33, D34, D35, D36, D37, D38, D39, D4, D40, D41, D42, D43, D44, D45, D46, D47, D48, D49, D5, D50, D51, D52, D53, D54, D55, D56, D57, D58, D59, D6, D60, D61, D62, D63, D7, D8, D9: D_ALT, symbol Device:D_ALT
- added RS1, RS11, RS12, RS13, RS14, RS15, RS16, RS17, RS18, RS19 (x2), RS2, RS20, RS21, RS23, RS24, RS25, RS26, RS27, RS28, RS29, RS3, RS30, RS31, RS32, RS33 (x2), RS34, RS35, RS36, RS37, RS38, RS39, RS4, RS40, RS41, RS42, RS43, RS44, RS45, RS46 (x2), RS47, RS49, RS5, RS50, RS51, RS52, RS53, RS54, RS55, RS56, RS57, RS58, RS59, RS6, RS60, RS61, RS62, RS63, RS7, RS8, RS9: 1k, symbol Device:R
- added SW1, SW10, SW11, SW12, SW13, SW14, SW15, SW16, SW17, SW18, SW19, SW2, SW20, SW21, SW22, SW23, SW24, SW25, SW26, SW27, SW28, SW29, SW3, SW30, SW31, SW32, SW33, SW34, SW35, SW36, SW37, SW38, SW39, SW4, SW40, SW41, SW42, SW43, SW44, SW45, SW46, SW47, SW48, SW49, SW5, SW50, SW51, SW52, SW53, SW54, SW55, SW56, SW57, SW58, SW59, SW6, SW60, SW61, SW62, SW63, SW7, SW8, SW9: KEY, symbol mykeyboard-rescue:KEY
Connections:
- new net: D1.1 (K), SW1.2
- new net: RS1.2, SW1.4
- new net: D2.1 (K), SW2.2
- new net: RS2.2, SW2.4
- new net: D3.1 (K), SW3.2
- new net: RS3.2, SW3.4
- new net: D4.1 (K), SW4.2
- new net: RS4.2, SW4.4
- new net: D5.1 (K), SW5.2
- new net: RS5.2, SW5.4
- new net: D6.1 (K), SW6.2
- new net: RS6.2, SW6.4
- new net: D7.1 (K), SW7.2
- new net: RS7.2, SW7.4
- new net: D8.1 (K), SW8.2
- new net: RS8.2, SW8.4
- new net: D9.1 (K), SW9.2
- new net: RS9.2, SW9.4
- new net: D10.1 (K), SW10.2
- new net: RS19.2, SW10.4
- new net: D11.1 (K), SW11.2
- new net: RS11.2, SW11.4
- new net: D12.1 (K), SW12.2
- new net: RS12.2, SW12.4
- new net: D13.1 (K), SW13.2
- new net: RS13.2, SW13.4
- new net: D14.1 (K), SW14.2
- new net: RS14.2, SW14.4
- new net: D15.1 (K), SW15.2
- new net: RS15.2, SW15.4
- new net: D16.1 (K), SW16.2
- new net: RS16.2, SW16.4
- new net: D17.1 (K), SW17.2
- new net: RS17.2, SW17.4
- new net: D18.1 (K), SW18.2
- new net: RS18.2, SW18.4
- new net: D19.1 (K), SW19.2
- new net: RS19.2, SW19.4
- new net: D20.1 (K), SW20.2
- new net: RS20.2, SW20.4
- new net: D21.1 (K), SW21.2
- new net: RS21.2, SW21.4
- new net: D22.1 (K), SW22.2
- new net: RS33.2, SW22.4
- new net: D23.1 (K), SW23.2
- new net: RS23.2, SW23.4
- new net: D24.1 (K), SW24.2
- new net: RS24.2, SW24.4
- new net: D25.1 (K), SW25.2
- new net: RS25.2, SW25.4
- new net: D26.1 (K), SW26.2
- new net: RS26.2, SW26.4
- new net: D27.1 (K), SW27.2
- new net: RS27.2, SW27.4
- new net: D28.1 (K), SW28.2
- new net: RS28.2, SW28.4
- new net: D29.1 (K), SW29.2
- new net: RS29.2, SW29.4
- new net: D30.1 (K), SW30.2
- new net: RS30.2, SW30.4
- new net: D31.1 (K), SW31.2
- new net: RS31.2, SW31.4
- new net: D32.1 (K), SW32.2
- new net: RS32.2, SW32.4
- new net: D33.1 (K), SW33.2
- new net: RS33.2, SW33.4
- new net: D34.1 (K), SW34.2
- new net: RS34.2, SW34.4
- new net: D35.1 (K), SW35.2
- new net: RS35.2, SW35.4
- new net: D36.1 (K), SW36.2
- new net: RS36.2, SW36.4
- new net: D37.1 (K), SW37.2
- new net: RS37.2, SW37.4
- new net: D38.1 (K), SW38.2
- new net: RS38.2, SW38.4
- new net: D39.1 (K), SW39.2
- new net: RS39.2, SW39.4
- new net: D40.1 (K), SW40.2
- new net: RS40.2, SW40.4
- new net: D41.1 (K), SW41.2
- new net: RS41.2, SW41.4
- new net: D42.1 (K), SW42.2
- new net: RS42.2, SW42.4
- new net: D43.1 (K), SW43.2
- new net: RS43.2, SW43.4
- new net: D44.1 (K), SW44.2
- new net: RS44.2, SW44.4
- new net: D45.1 (K), SW45.2
- new net: RS45.2, SW45.4
- new net: D46.1 (K), SW46.2
- new net: RS46.2, SW46.4
- new net: D47.1 (K), SW47.2
- new net: RS47.2, SW47.4
- new net: D48.1 (K), SW48.2
- new net: RS46.2, SW48.4
- new net: D49.1 (K), SW49.2
- new net: RS49.2, SW49.4
- new net: D50.1 (K), SW50.2
- new net: RS50.2, SW50.4
- new net: D51.1 (K), SW51.2
- new net: RS51.2, SW51.4
- new net: D52.1 (K), SW52.2
- new net: RS52.2, SW52.4
- new net: D53.1 (K), SW53.2
- new net: RS53.2, SW53.4
- new net: D54.1 (K), SW54.2
- new net: RS54.2, SW54.4
- new net: D55.1 (K), SW55.2
- new net: RS55.2, SW55.4
- new net: D56.1 (K), SW56.2
- new net: RS56.2, SW56.4
- new net: D57.1 (K), SW57.2
- new net: RS57.2, SW57.4
- new net: D58.1 (K), SW58.2
- new net: RS58.2, SW58.4
- new net: D59.1 (K), SW59.2
- new net: RS59.2, SW59.4
- new net: D61.1 (K), SW61.2
- new net: RS61.2, SW61.4
- new net: D62.1 (K), SW62.2
- new net: RS62.2, SW62.4
- new net: D63.1 (K), SW63.2
- new net: RS63.2, SW63.4
- new net: D60.1 (K), SW60.2
- new net: RS60.2, SW60.4
- new net col1: SW1.1, SW15.1, SW29.1, SW43.1, SW57.1
- new net col10: SW10.1, SW24.1, SW38.1, SW52.1
- new net col11: RS11.1, RS25.1, RS39.1, RS53.1, SW11.1, SW25.1, SW39.1, SW53.1
- new net col12: SW12.1, SW26.1, SW40.1, SW54.1, SW61.1
- new net col13: SW13.1, SW27.1, SW41.1, SW55.1, SW62.1
- new net col14: SW14.1, SW28.1, SW42.1, SW56.1, SW63.1
- new net col2: SW16.1, SW2.1, SW30.1, SW44.1, SW58.1
- new net col3: SW17.1, SW3.1, SW31.1, SW45.1, SW59.1
- new net col4: SW18.1, SW32.1, SW4.1, SW46.1
- new net col5: SW19.1, SW33.1, SW47.1, SW5.1
- new net col6: SW20.1, SW34.1, SW48.1, SW6.1
- new net col7: SW21.1, SW35.1, SW49.1, SW7.1
- new net col8: SW22.1, SW36.1, SW50.1, SW60.1, SW8.1
- new net col9: SW23.1, SW37.1, SW51.1, SW9.1
- new net lcol1: RS1.1, RS15.1, RS29.1, RS43.1, RS57.1
- new net lcol10: RS19.1, RS24.1, RS38.1, RS52.1
- new net lcol12: RS12.1, RS26.1, RS40.1, RS54.1, RS61.1
- new net lcol13: RS13.1, RS27.1, RS41.1, RS55.1, RS62.1
- new net lcol14: RS14.1, RS28.1, RS42.1, RS56.1, RS63.1
- new net lcol2: RS16.1, RS2.1, RS30.1, RS44.1, RS58.1
- new net lcol3: RS17.1, RS3.1, RS31.1, RS45.1, RS59.1
- new net lcol4: RS18.1, RS32.1, RS4.1, RS46.1
- new net lcol5: RS19.1, RS33.1, RS47.1, RS5.1
- new net lcol6: RS20.1, RS34.1, RS46.1, RS6.1
- new net lcol7: RS21.1, RS35.1, RS49.1, RS7.1
- new net lcol8: RS50.1, RS60.1, RS8.1
- new net lcol9: RS23.1, RS37.1, RS51.1, RS9.1
- new net lrow1: SW1.3, SW10.3, SW11.3, SW12.3, SW13.3, SW14.3, SW2.3, SW3.3, SW4.3, SW5.3, SW6.3, SW7.3, SW8.3, SW9.3
- new net lrow2: SW15.3, SW16.3, SW17.3, SW18.3, SW19.3, SW20.3, SW21.3, SW22.3, SW23.3, SW24.3, SW25.3, SW26.3, SW27.3, SW28.3
- new net lrow3: SW29.3, SW30.3, SW31.3, SW32.3, SW33.3, SW34.3, SW35.3, SW36.3, SW37.3, SW38.3, SW39.3, SW40.3, SW41.3, SW42.3
- new net lrow4: SW43.3, SW44.3, SW45.3, SW46.3, SW47.3, SW48.3, SW49.3, SW50.3, SW51.3, SW52.3, SW53.3, SW54.3, SW55.3, SW56.3
- new net lrow5: SW57.3, SW58.3, SW59.3, SW60.3, SW61.3, SW62.3, SW63.3
- new net row1: D1.2 (A), D10.2 (A), D11.2 (A), D12.2 (A), D13.2 (A), D14.2 (A), D2.2 (A), D3.2 (A), D4.2 (A), D5.2 (A), D6.2 (A), D7.2 (A), D8.2 (A), D9.2 (A)
- new net row2: D15.2 (A), D16.2 (A), D17.2 (A), D18.2 (A), D19.2 (A), D20.2 (A), D21.2 (A), D22.2 (A), D23.2 (A), D24.2 (A), D25.2 (A), D26.2 (A), D27.2 (A), D28.2 (A)
- new net row3: D29.2 (A), D30.2 (A), D31.2 (A), D32.2 (A), D33.2 (A), D34.2 (A), D35.2 (A), D36.2 (A), D37.2 (A), D38.2 (A), D39.2 (A), D40.2 (A), D41.2 (A), D42.2 (A)
- new net row4: D43.2 (A), D44.2 (A), D45.2 (A), D46.2 (A), D47.2 (A), D48.2 (A), D49.2 (A), D50.2 (A), D51.2 (A), D52.2 (A), D53.2 (A), D54.2 (A), D55.2 (A), D56.2 (A)
- new net row5: D57.2 (A), D58.2 (A), D59.2 (A), D60.2 (A), D61.2 (A), D62.2 (A), D63.2 (A)

Commit message: gogogogit pull!
Parts:
- added D45, D50: D_ALT, Diode_SMD:D_0805_2012Metric_Pad1.15x1.40mm_HandSolder, symbol Device:D_ALT
- added RS45, RS50: 1k, Resistor_SMD:R_0805_2012Metric_Pad1.15x1.40mm_HandSolder, symbol Device:R
- added SW46, SW51: KEY, mykeyboard:MX_LED, symbol mykeyboard-rescue:KEY
- D1, D54: footprint (none) -> Diode_SMD:D_0805_2012Metric_Pad1.15x1.40mm_HandSolder
- D10: renamed from D58; footprint (none) -> Diode_SMD:D_0805_2012Metric_Pad1.15x1.40mm_HandSolder
- D11: renamed from D3; footprint (none) -> Diode_SMD:D_0805_2012Metric_Pad1.15x1.40mm_HandSolder
- D12: renamed from D17; footprint (none) -> Diode_SMD:D_0805_2012Metric_Pad1.15x1.40mm_HandSolder
- D13: renamed from D31; footprint (none) -> Diode_SMD:D_0805_2012Metric_Pad1.15x1.40mm_HandSolder
- D14: renamed from D45; footprint (none) -> Diode_SMD:D_0805_2012Metric_Pad1.15x1.40mm_HandSolder
- D15: renamed from D59; footprint (none) -> Diode_SMD:D_0805_2012Metric_Pad1.15x1.40mm_HandSolder
- D16: renamed from D4; footprint (none) -> Diode_SMD:D_0805_2012Metric_Pad1.15x1.40mm_HandSolder
- D17: renamed from D18; footprint (none) -> Diode_SMD:D_0805_2012Metric_Pad1.15x1.40mm_HandSolder
- D18: renamed from D32; footprint (none) -> Diode_SMD:D_0805_2012Metric_Pad1.15x1.40mm_HandSolder
- D19: renamed from D46; footprint (none) -> Diode_SMD:D_0805_2012Metric_Pad1.15x1.40mm_HandSolder
- D2: renamed from D15; footprint (none) -> Diode_SMD:D_0805_2012Metric_Pad1.15x1.40mm_HandSolder
- D20: renamed from D5; footprint (none) -> Diode_SMD:D_0805_2012Metric_Pad1.15x1.40mm_HandSolder
- D21: renamed from D19; footprint (none) -> Diode_SMD:D_0805_2012Metric_Pad1.15x1.40mm_HandSolder
- D22: renamed from D33; footprint (none) -> Diode_SMD:D_0805_2012Metric_Pad1.15x1.40mm_HandSolder
- D23: renamed from D47; footprint (none) -> Diode_SMD:D_0805_2012Metric_Pad1.15x1.40mm_HandSolder
- D24: renamed from D6; footprint (none) -> Diode_SMD:D_0805_2012Metric_Pad1.15x1.40mm_HandSolder
- D25: renamed from D20; footprint (none) -> Diode_SMD:D_0805_2012Metric_Pad1.15x1.40mm_HandSolder
- D26: renamed from D34; footprint (none) -> Diode_SMD:D_0805_2012Metric_Pad1.15x1.40mm_HandSolder
- D27: renamed from D48; footprint (none) -> Diode_SMD:D_0805_2012Metric_Pad1.15x1.40mm_HandSolder
- D28: renamed from D7; footprint (none) -> Diode_SMD:D_0805_2012Metric_Pad1.15x1.40mm_HandSolder
- D29: renamed from D21; footprint (none) -> Diode_SMD:D_0805_2012Metric_Pad1.15x1.40mm_HandSolder
- D3: renamed from D29; footprint (none) -> Diode_SMD:D_0805_2012Metric_Pad1.15x1.40mm_HandSolder
- D30: renamed from D35; footprint (none) -> Diode_SMD:D_0805_2012Metric_Pad1.15x1.40mm_HandSolder
- D31: renamed from D49; footprint (none) -> Diode_SMD:D_0805_2012Metric_Pad1.15x1.40mm_HandSolder
- D32: renamed from D8; footprint (none) -> Diode_SMD:D_0805_2012Metric_Pad1.15x1.40mm_HandSolder
- D33: renamed from D22; footprint (none) -> Diode_SMD:D_0805_2012Metric_Pad1.15x1.40mm_HandSolder
- D34: renamed from D36; footprint (none) -> Diode_SMD:D_0805_2012Metric_Pad1.15x1.40mm_HandSolder
- D35: renamed from D50; footprint (none) -> Diode_SMD:D_0805_2012Metric_Pad1.15x1.40mm_HandSolder
- D36: renamed from D60; footprint (none) -> Diode_SMD:D_0805_2012Metric_Pad1.15x1.40mm_HandSolder
- D37: renamed from D9; footprint (none) -> Diode_SMD:D_0805_2012Metric_Pad1.15x1.40mm_HandSolder
- D38: renamed from D23; footprint (none) -> Diode_SMD:D_0805_2012Metric_Pad1.15x1.40mm_HandSolder
- D39: renamed from D37; footprint (none) -> Diode_SMD:D_0805_2012Metric_Pad1.15x1.40mm_HandSolder
- D4: renamed from D43; footprint (none) -> Diode_SMD:D_0805_2012Metric_Pad1.15x1.40mm_HandSolder
- D40: renamed from D51; footprint (none) -> Diode_SMD:D_0805_2012Metric_Pad1.15x1.40mm_HandSolder
- D41: renamed from D10; footprint (none) -> Diode_SMD:D_0805_2012Metric_Pad1.15x1.40mm_HandSolder
- D42: renamed from D24; footprint (none) -> Diode_SMD:D_0805_2012Metric_Pad1.15x1.40mm_HandSolder
- D43: renamed from D38; footprint (none) -> Diode_SMD:D_0805_2012Metric_Pad1.15x1.40mm_HandSolder
- D44: renamed from D52; footprint (none) -> Diode_SMD:D_0805_2012Metric_Pad1.15x1.40mm_HandSolder
- D46: renamed from D11; footprint (none) -> Diode_SMD:D_0805_2012Metric_Pad1.15x1.40mm_HandSolder
- D47: renamed from D25; footprint (none) -> Diode_SMD:D_0805_2012Metric_Pad1.15x1.40mm_HandSolder
- D48: renamed from D39; footprint (none) -> Diode_SMD:D_0805_2012Metric_Pad1.15x1.40mm_HandSolder
- D49: renamed from D53; footprint (none) -> Diode_SMD:D_0805_2012Metric_Pad1.15x1.40mm_HandSolder
- D5: renamed from D57; footprint (none) -> Diode_SMD:D_0805_2012Metric_Pad1.15x1.40mm_HandSolder
- D51: renamed from D12; footprint (none) -> Diode_SMD:D_0805_2012Metric_Pad1.15x1.40mm_HandSolder
- D52: renamed from D26; footprint (none) -> Diode_SMD:D_0805_2012Metric_Pad1.15x1.40mm_HandSolder
- D53: renamed from D40; footprint (none) -> Diode_SMD:D_0805_2012Metric_Pad1.15x1.40mm_HandSolder
- D55: renamed from D61; footprint (none) -> Diode_SMD:D_0805_2012Metric_Pad1.15x1.40mm_HandSolder
- D56: renamed from D13; footprint (none) -> Diode_SMD:D_0805_2012Metric_Pad1.15x1.40mm_HandSolder
- D57: renamed from D27; footprint (none) -> Diode_SMD:D_0805_2012Metric_Pad1.15x1.40mm_HandSolder
- D58: renamed from D41; footprint (none) -> Diode_SMD:D_0805_2012Metric_Pad1.15x1.40mm_HandSolder
- D59: renamed from D55; footprint (none) -> Diode_SMD:D_0805_2012Metric_Pad1.15x1.40mm_HandSolder
- D6: renamed from D2; footprint (none) -> Diode_SMD:D_0805_2012Metric_Pad1.15x1.40mm_HandSolder
- D60: renamed from D62; footprint (none) -> Diode_SMD:D_0805_2012Metric_Pad1.15x1.40mm_HandSolder
- D61: renamed from D14; footprint (none) -> Diode_SMD:D_0805_2012Metric_Pad1.15x1.40mm_HandSolder
- D62: renamed from D28; footprint (none) -> Diode_SMD:D_0805_2012Metric_Pad1.15x1.40mm_HandSolder
- D63: renamed from D42; footprint (none) -> Diode_SMD:D_0805_2012Metric_Pad1.15x1.40mm_HandSolder
- D64: renamed from D56; footprint (none) -> Diode_SMD:D_0805_2012Metric_Pad1.15x1.40mm_HandSolder
- D65: renamed from D63; footprint (none) -> Diode_SMD:D_0805_2012Metric_Pad1.15x1.40mm_HandSolder
- D7: renamed from D16; footprint (none) -> Diode_SMD:D_0805_2012Metric_Pad1.15x1.40mm_HandSolder
- D8: renamed from D30; footprint (none) -> Diode_SMD:D_0805_2012Metric_Pad1.15x1.40mm_HandSolder
- D9: renamed from D44; footprint (none) -> Diode_SMD:D_0805_2012Metric_Pad1.15x1.40mm_HandSolder
- RS1, RS33, RS54: footprint (none) -> Resistor_SMD:R_0805_2012Metric_Pad1.15x1.40mm_HandSolder
- RS10: renamed from RS58; footprint (none) -> Resistor_SMD:R_0805_2012Metric_Pad1.15x1.40mm_HandSolder
- RS11: renamed from RS3; footprint (none) -> Resistor_SMD:R_0805_2012Metric_Pad1.15x1.40mm_HandSolder
- RS12: renamed from RS17; footprint (none) -> Resistor_SMD:R_0805_2012Metric_Pad1.15x1.40mm_HandSolder
- RS13: renamed from RS31; footprint (none) -> Resistor_SMD:R_0805_2012Metric_Pad1.15x1.40mm_HandSolder
- RS14: renamed from RS45; footprint (none) -> Resistor_SMD:R_0805_2012Metric_Pad1.15x1.40mm_HandSolder
- RS15: renamed from RS59; footprint (none) -> Resistor_SMD:R_0805_2012Metric_Pad1.15x1.40mm_HandSolder
- RS16: renamed from RS4; footprint (none) -> Resistor_SMD:R_0805_2012Metric_Pad1.15x1.40mm_HandSolder
- RS17: renamed from RS18; footprint (none) -> Resistor_SMD:R_0805_2012Metric_Pad1.15x1.40mm_HandSolder
- RS18: renamed from RS32; footprint (none) -> Resistor_SMD:R_0805_2012Metric_Pad1.15x1.40mm_HandSolder
- RS19, RS27: renamed from RS46; footprint (none) -> Resistor_SMD:R_0805_2012Metric_Pad1.15x1.40mm_HandSolder
- RS2: renamed from RS15; footprint (none) -> Resistor_SMD:R_0805_2012Metric_Pad1.15x1.40mm_HandSolder
- RS20: renamed from RS5; footprint (none) -> Resistor_SMD:R_0805_2012Metric_Pad1.15x1.40mm_HandSolder
- RS21, RS41: renamed from RS19; footprint (none) -> Resistor_SMD:R_0805_2012Metric_Pad1.15x1.40mm_HandSolder
- RS22: renamed from RS33; footprint (none) -> Resistor_SMD:R_0805_2012Metric_Pad1.15x1.40mm_HandSolder
- RS23: renamed from RS47; footprint (none) -> Resistor_SMD:R_0805_2012Metric_Pad1.15x1.40mm_HandSolder
- RS24: renamed from RS6; footprint (none) -> Resistor_SMD:R_0805_2012Metric_Pad1.15x1.40mm_HandSolder
- RS25: renamed from RS20; footprint (none) -> Resistor_SMD:R_0805_2012Metric_Pad1.15x1.40mm_HandSolder
- RS26: renamed from RS34; footprint (none) -> Resistor_SMD:R_0805_2012Metric_Pad1.15x1.40mm_HandSolder
- RS28: renamed from RS7; footprint (none) -> Resistor_SMD:R_0805_2012Metric_Pad1.15x1.40mm_HandSolder
- RS29: renamed from RS21; footprint (none) -> Resistor_SMD:R_0805_2012Metric_Pad1.15x1.40mm_HandSolder
- RS3: renamed from RS29; footprint (none) -> Resistor_SMD:R_0805_2012Metric_Pad1.15x1.40mm_HandSolder
- RS30: renamed from RS35; footprint (none) -> Resistor_SMD:R_0805_2012Metric_Pad1.15x1.40mm_HandSolder
- RS31: renamed from RS49; footprint (none) -> Resistor_SMD:R_0805_2012Metric_Pad1.15x1.40mm_HandSolder
- RS32: renamed from RS8; footprint (none) -> Resistor_SMD:R_0805_2012Metric_Pad1.15x1.40mm_HandSolder
- RS34: renamed from RS36; footprint (none) -> Resistor_SMD:R_0805_2012Metric_Pad1.15x1.40mm_HandSolder
- RS35: renamed from RS50; footprint (none) -> Resistor_SMD:R_0805_2012Metric_Pad1.15x1.40mm_HandSolder
- RS36: renamed from RS60; footprint (none) -> Resistor_SMD:R_0805_2012Metric_Pad1.15x1.40mm_HandSolder
- RS37: renamed from RS9; footprint (none) -> Resistor_SMD:R_0805_2012Metric_Pad1.15x1.40mm_HandSolder
- RS38: renamed from RS23; footprint (none) -> Resistor_SMD:R_0805_2012Metric_Pad1.15x1.40mm_HandSolder
- RS39: renamed from RS37; footprint (none) -> Resistor_SMD:R_0805_2012Metric_Pad1.15x1.40mm_HandSolder
- RS4: renamed from RS43; footprint (none) -> Resistor_SMD:R_0805_2012Metric_Pad1.15x1.40mm_HandSolder
- RS40: renamed from RS51; footprint (none) -> Resistor_SMD:R_0805_2012Metric_Pad1.15x1.40mm_HandSolder
- RS42: renamed from RS24; footprint (none) -> Resistor_SMD:R_0805_2012Metric_Pad1.15x1.40mm_HandSolder
- RS43: renamed from RS38; footprint (none) -> Resistor_SMD:R_0805_2012Metric_Pad1.15x1.40mm_HandSolder
- RS44: renamed from RS52; footprint (none) -> Resistor_SMD:R_0805_2012Metric_Pad1.15x1.40mm_HandSolder
- RS46: renamed from RS11; footprint (none) -> Resistor_SMD:R_0805_2012Metric_Pad1.15x1.40mm_HandSolder
- RS47: renamed from RS25; footprint (none) -> Resistor_SMD:R_0805_2012Metric_Pad1.15x1.40mm_HandSolder
- RS48: renamed from RS39; footprint (none) -> Resistor_SMD:R_0805_2012Metric_Pad1.15x1.40mm_HandSolder
- RS49: renamed from RS53; footprint (none) -> Resistor_SMD:R_0805_2012Metric_Pad1.15x1.40mm_HandSolder
- RS5: renamed from RS57; footprint (none) -> Resistor_SMD:R_0805_2012Metric_Pad1.15x1.40mm_HandSolder
- RS51: renamed from RS12; footprint (none) -> Resistor_SMD:R_0805_2012Metric_Pad1.15x1.40mm_HandSolder
- RS52: renamed from RS26; footprint (none) -> Resistor_SMD:R_0805_2012Metric_Pad1.15x1.40mm_HandSolder
- RS53: renamed from RS40; footprint (none) -> Resistor_SMD:R_0805_2012Metric_Pad1.15x1.40mm_HandSolder
- RS55: renamed from RS61; footprint (none) -> Resistor_SMD:R_0805_2012Metric_Pad1.15x1.40mm_HandSolder
- RS56: renamed from RS13; footprint (none) -> Resistor_SMD:R_0805_2012Metric_Pad1.15x1.40mm_HandSolder
- RS57: renamed from RS27; footprint (none) -> Resistor_SMD:R_0805_2012Metric_Pad1.15x1.40mm_HandSolder
- RS58: renamed from RS41; footprint (none) -> Resistor_SMD:R_0805_2012Metric_Pad1.15x1.40mm_HandSolder
- RS59: renamed from RS55; footprint (none) -> Resistor_SMD:R_0805_2012Metric_Pad1.15x1.40mm_HandSolder
- RS6: renamed from RS2; footprint (none) -> Resistor_SMD:R_0805_2012Metric_Pad1.15x1.40mm_HandSolder
- RS60: renamed from RS62; footprint (none) -> Resistor_SMD:R_0805_2012Metric_Pad1.15x1.40mm_HandSolder
- RS61: renamed from RS14; footprint (none) -> Resistor_SMD:R_0805_2012Metric_Pad1.15x1.40mm_HandSolder
- RS62: renamed from RS28; footprint (none) -> Resistor_SMD:R_0805_2012Metric_Pad1.15x1.40mm_HandSolder
- RS63: renamed from RS42; footprint (none) -> Resistor_SMD:R_0805_2012Metric_Pad1.15x1.40mm_HandSolder
- RS64: renamed from RS56; footprint (none) -> Resistor_SMD:R_0805_2012Metric_Pad1.15x1.40mm_HandSolder
- RS65: renamed from RS63; footprint (none) -> Resistor_SMD:R_0805_2012Metric_Pad1.15x1.40mm_HandSolder
- RS7: renamed from RS16; footprint (none) -> Resistor_SMD:R_0805_2012Metric_Pad1.15x1.40mm_HandSolder
- RS8: renamed from RS30; footprint (none) -> Resistor_SMD:R_0805_2012Metric_Pad1.15x1.40mm_HandSolder
- RS9: renamed from RS44; footprint (none) -> Resistor_SMD:R_0805_2012Metric_Pad1.15x1.40mm_HandSolder
- SW10: renamed from SW44; footprint (none) -> mykeyboard:MX_LED
- SW11: renamed from SW58; footprint (none) -> mykeyboard:MX_LED
- SW12: renamed from SW3; footprint (none) -> mykeyboard:MX_LED
- SW13: renamed from SW17; footprint (none) -> mykeyboard:MX_LED
- SW14: renamed from SW31; footprint (none) -> mykeyboard:MX_LED
- SW15: renamed from SW45; footprint (none) -> mykeyboard:MX_LED
- SW16: renamed from SW59; footprint (none) -> mykeyboard:MX_LED
- SW17: renamed from SW4; footprint (none) -> mykeyboard:MX_LED
- SW18: footprint (none) -> mykeyboard:MX_LED
- SW19: renamed from SW32; footprint (none) -> mykeyboard:MX_LED
- SW2: renamed from SW1; footprint (none) -> mykeyboard:MX_LED
- SW20: renamed from SW46; footprint (none) -> mykeyboard:MX_LED
- SW21: renamed from SW5; footprint (none) -> mykeyboard:MX_LED
- SW22: renamed from SW19; footprint (none) -> mykeyboard:MX_LED
- SW23: renamed from SW33; footprint (none) -> mykeyboard:MX_LED
- SW24: renamed from SW47; footprint (none) -> mykeyboard:MX_LED
- SW25: renamed from SW6; footprint (none) -> mykeyboard:MX_LED
- SW26: renamed from SW20; footprint (none) -> mykeyboard:MX_LED
- SW27: renamed from SW34; footprint (none) -> mykeyboard:MX_LED
- SW28: renamed from SW48; footprint (none) -> mykeyboard:MX_LED
- SW29: renamed from SW7; footprint (none) -> mykeyboard:MX_LED
- SW3: renamed from SW15; footprint (none) -> mykeyboard:MX_LED
- SW30: renamed from SW21; footprint (none) -> mykeyboard:MX_LED
- SW31: renamed from SW35; footprint (none) -> mykeyboard:MX_LED
- SW32: renamed from SW49; footprint (none) -> mykeyboard:MX_LED
- SW33: renamed from SW8; footprint (none) -> mykeyboard:MX_LED
- SW34: renamed from SW22; footprint (none) -> mykeyboard:MX_LED
- SW35: renamed from SW36; footprint (none) -> mykeyboard:MX_LED
- SW36: renamed from SW50; footprint (none) -> mykeyboard:MX_LED
- SW37: renamed from SW60; footprint (none) -> mykeyboard:MX_LED
- SW38: renamed from SW9; footprint (none) -> mykeyboard:MX_LED
- SW39: renamed from SW23; footprint (none) -> mykeyboard:MX_LED
- SW4: renamed from SW29; footprint (none) -> mykeyboard:MX_LED
- SW40: renamed from SW37; footprint (none) -> mykeyboard:MX_LED
- SW41: renamed from SW51; footprint (none) -> mykeyboard:MX_LED
- SW42: renamed from SW10; footprint (none) -> mykeyboard:MX_LED
- SW43: renamed from SW24; footprint (none) -> mykeyboard:MX_LED
- SW44: renamed from SW38; footprint (none) -> mykeyboard:MX_LED
- SW45: renamed from SW52; footprint (none) -> mykeyboard:MX_LED
- SW47: renamed from SW11; footprint (none) -> mykeyboard:MX_LED
- SW48: renamed from SW25; footprint (none) -> mykeyboard:MX_LED
- SW49: renamed from SW39; footprint (none) -> mykeyboard:MX_LED
- SW5: renamed from SW43; footprint (none) -> mykeyboard:MX_LED
- SW50: renamed from SW53; footprint (none) -> mykeyboard:MX_LED
- SW52: renamed from SW12; footprint (none) -> mykeyboard:MX_LED
- SW53: renamed from SW26; footprint (none) -> mykeyboard:MX_LED
- SW54: renamed from SW40; footprint (none) -> mykeyboard:MX_LED
- SW55: renamed from SW54; footprint (none) -> mykeyboard:MX_LED
- SW56: renamed from SW61; footprint (none) -> mykeyboard:MX_LED
- SW57: renamed from SW13; footprint (none) -> mykeyboard:MX_LED
- SW58: renamed from SW27; footprint (none) -> mykeyboard:MX_LED
- SW59: renamed from SW41; footprint (none) -> mykeyboard:MX_LED
- SW6: renamed from SW57; footprint (none) -> mykeyboard:MX_LED
- SW60: renamed from SW55; footprint (none) -> mykeyboard:MX_LED
- SW61: renamed from SW62; footprint (none) -> mykeyboard:MX_LED
- SW62: renamed from SW14; footprint (none) -> mykeyboard:MX_LED
- SW63: renamed from SW28; footprint (none) -> mykeyboard:MX_LED
- SW64: renamed from SW42; footprint (none) -> mykeyboard:MX_LED
- SW65: renamed from SW56; footprint (none) -> mykeyboard:MX_LED
- SW66: renamed from SW63; footprint (none) -> mykeyboard:MX_LED
- SW7: renamed from SW2; footprint (none) -> mykeyboard:MX_LED
- SW8: renamed from SW16; footprint (none) -> mykeyboard:MX_LED
- SW9: renamed from SW30; footprint (none) -> mykeyboard:MX_LED
Connections:
- net col10: now also SW46.1
- net col11: now also RS50.1
- net col6: now also SW37.1
- net col8: no longer SW37.1
- net lcol10: now also RS45.1
- net lcol6: now also RS36.1
- net lcol8: now also RS33.1, RS34.1; no longer RS36.1
- net row5: now also D45.2 (A), D50.2 (A)
- new net: D50.1 (K), SW51.2
- new net: RS50.2, SW51.4
- new net: D45.1 (K), SW46.2
- new net: RS45.2, SW46.4
Other:
- moved on the sheet: D36, RS36, SW37

Commit message: junk,but still a good prove.
Connections:
- net col11: now also SW51.1; no longer RS46.1, RS47.1, RS48.1, RS49.1, RS50.1
- new net lcol11: RS46.1, RS47.1, RS48.1, RS49.1, RS50.1
Changed lines of the file:
@@
 lcol10
 Text GLabel 8700 950  1    50   Input ~ 0
-col11
+lcol11
 Text GLabel 9400 950  1    50   Input ~ 0
 lcol12
@@
 Wire Wire Line
 	8800 5450 9500 5450
+Wire Wire Line
+	8350 6000 8350 5000
+Connection ~ 8350 5000
 $EndSCHEMATC
