File: mykeyboard/mykeyboard.kicad_pcb (KiCad board)
At the start: 2 copper layers, 255 parts, among them J1 USB_A, J2 USB_A, J3 USB_A, J4 USB_B, J5 Conn_01x08_Male, J6 Conn_01x24_Female, SW10 KEY, SW11 KEY, SW12 KEY, SW13 KEY, SW14 KEY, SW15 KEY, SW16 KEY, SW17 KEY, SW18 KEY, SW19 KEY, SW2 KEY, SW20 KEY, SW21 KEY, SW22 KEY, SW23 KEY, SW24 KEY, SW25 KEY, SW26 KEY, SW27 KEY, SW28 KEY, SW29 KEY, SW3 KEY, SW30 KEY, SW31 KEY, SW32 KEY, SW33 KEY, SW34 KEY, SW35 KEY, SW36 KEY, SW37 KEY, SW38 KEY, SW39 KEY, SW4 KEY, SW40 KEY, SW41 KEY, SW42 KEY, SW43 KEY, SW44 KEY, SW45 KEY, SW46 KEY, SW47 KEY, SW48 KEY, SW49 KEY, SW5 KEY, SW50 KEY, SW51 KEY, SW52 KEY, SW53 KEY, SW54 KEY, SW55 KEY, SW56 KEY, SW57 KEY, SW58 KEY, SW59 KEY, SW6 KEY, SW60 KEY, SW61 KEY, SW62 KEY, SW63 KEY, SW64 KEY, SW65 KEY, SW66 KEY, SW7 KEY, SW8 KEY, SW9 KEY, U1 TLV1117-33, U2 GL850A, U3 ATmega32U4-AU, X1 3325-12MHz, X2 3325-16MHz

Commit message: junk,but still a good prove.
Parts:
- added SW1: SW_SPST, mykeyboard:SW, F.Cu at (97.8, 47.0)
- C10, C4, C5, C8, C9, J1, J2, J3, J4, R15, R17, R18, R19, R2, R3, R6, RS1, RS10, RS11, RS12, RS13, RS14, RS15, RS16, RS17, RS18, RS19, RS2, RS20, RS21, RS22, RS23, RS24, RS25, RS26, RS27, RS28, RS29, RS3, RS30, RS31, RS32, RS33, RS34, RS35, RS36, RS37, RS38, RS39, RS4, RS40, RS41, RS42, RS43, RS44, RS45, RS46, RS47, RS48, RS49, RS50, RS51, RS52, RS53, RS54, RS55, RS56, RS57, RS58, RS59, RS6, RS60, RS61, RS62, RS63, RS64, RS65, RS7, RS8, RS9, U3, X1, X2: moved to B.Cu
- D10, D15, D5: moved to F.Cu
- moved J1 449.7 mm to (306.8, 49.5), turned to 270 degrees
- moved R13 423.6 mm to (290.6, 42.7), turned to 45 degrees
- moved X1 414.3 mm to (280.6, 11.1), turned to 180 degrees
- moved R5 400.3 mm to (295.9, 47.8), turned to 45 degrees
- moved R1 399.7 mm to (290.3, 52.6), turned to 45 degrees
- moved R2 394.2 mm to (293.1, 50.5), turned to 180 degrees
- moved R3 394.1 mm to (297.2, 48.5)
- moved R7 391.8 mm to (295.9, 42.4), turned to 45 degrees
- moved R4 388.7 mm to (295.9, 52.6), turned to 45 degrees
- moved U2 388.1 mm to (280.2, 46.7), turned to 315 degrees
- moved C7 385.9 mm to (256.0, 42.7), turned to 90 degrees
- moved C2 383.6 mm to (290.3, 47.8), turned to 225 degrees
- moved C14 383.2 mm to (270.8, 45.6), turned to 270 degrees
- moved C13 383.0 mm to (267.2, 45.6), turned to 270 degrees
- moved C4 380.8 mm to (276.6, 19.6), turned to 90 degrees
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Connections:
- RS46 pad 1: col11 -> lcol11
- RS47 pad 1: col11 -> lcol11
- RS48 pad 1: col11 -> lcol11
- RS49 pad 1: col11 -> lcol11
- RS50 pad 1: col11 -> lcol11
- SW51 pad 1: Net-(SW51-Pad1) -> col11
Routing:
- net row3: track 0.00 -> 406.1 mm
- net row4: track 0.00 -> 302.6 mm, vias 0 -> 2
- net lrow3: track 0.00 -> 295.2 mm, vias 0 -> 2
- net row1: track 0.00 -> 275.0 mm
- net lrow4: track 0.00 -> 274.3 mm, vias 0 -> 1
- net row2: track 0.00 -> 270.5 mm
- net row5: track 0.00 -> 261.0 mm
- net lrow1: track 0.00 -> 254.3 mm
- net lrow2: track 0.00 -> 253.9 mm
- net lrow5: track 0.00 -> 241.8 mm
- net lcol13: track 0.00 -> 237.9 mm
- net col2: track 0.00 -> 152.6 mm
- net lcol6: track 0.00 -> 150.1 mm
- net lcol2: track 0.00 -> 149.4 mm
- net col6: track 0.00 -> 114.1 mm
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Other:
- net class SW added: clearance 0.254, trace_width 0.381, via_dia 0.762, via_drill 0.508
