File: mykeyboard/mykeyboard.sch (KiCad schematic (older format))
At the start: 2 parts

Commit message: try to select PATH
Parts:
- removed U?: GL850A, symbol Switch:GL850A
Changed lines of the file:
@@
 EESchema Schematic File Version 4
+LIBS:mykeyboard-cache
 EELAYER 26 0
 EELAYER END
@@
 $EndDescr
 $Comp
-L Switch:GL850A U?
-U 1 1 5BE85F64
-P 3000 4200
-F 0 "U?" H 2975 5465 50  0000 C CNN
-F 1 "GL850A" H 2975 5374 50  0000 C CNN
-F 2 "" H 2300 5400 50  0001 C CNN
-F 3 "" H 2300 5400 50  0001 C CNN
-	1    3000 4200
-	1    0    0    -1
-$EndComp
-$Comp
 L MCU_Microchip_ATmega:ATmega32U4-AU U?

Commit message: 1112,gogogo
Parts:
- added C1, C3: 10u, symbol Device:CP1
- added C10, C11, C12, C18, C19, C2, C4, C5, C6, C7, C8, C9: 104, symbol Device:C
- added C13, C14, C15, C16: 22p, symbol Device:C
- added DF1, DF2, DF3, DF4: 0603G, symbol Device:LED_Small
- added FB1, FB2: ~, symbol Device:L
- added J1: USB_B, symbol Connector:USB_B
- added J2, J3, J4: USB_A, symbol Connector:USB_A
- added J5: Conn_01x24_Female, symbol Connector:Conn_01x24_Female
- added J?: Conn_01x08_Male, symbol Connector:Conn_01x08_Male
- added R1, R10, R11, R12, R16, R2, R5, R6, R7, R8, R9: 22, symbol Device:R
- added R13, R14, R15, R17: 100k, symbol Device:R
- added R18: 680, symbol Device:R
- added R19: 10k, symbol Device:R
- added R20, R21, R22, R23: 1k, symbol Device:R
- added R3, R4: 1M, symbol Device:R
- added SW0: SW_SPST, symbol Switch:SW_SPST
- added U0: TLV1117-33, symbol Regulator_Linear:TLV1117-33
- added U1: GL850A, symbol mykeyboard-rescue:GL850A-mykeyboardlibs
- added X1: 3325-16MHz, symbol mykeyboard-rescue:3325-16MHz-mykeyboardlibs
- added X2: 3325-12MHz, symbol mykeyboard-rescue:3325-12MHz-mykeyboardlibs
- gave numbers to parts that had none: 1
Connections:
- net col3: now reaches U2.1 (PE6)
- net caps_led: now reaches U2.10 (PB2)
- net caps_led: now also J?.4 (Pin_4)
- net col14: now reaches U2.11 (PB3)
- net col14: now also U2.32 (PC7), J?.3 (Pin_3)
- net col9: now reaches U2.12 (PB7)
- net RESET2#: now reaches U2.13 (~RESET)
- net RESET2#: now also J?.7 (Pin_7), R16.2, SW0.1 (A)
- net VCC: now reaches U2.14 (VCC), U2.34 (VCC)
- net VCC: now also U2.2 (UVCC), U2.24 (AVCC), U2.44 (AVCC), U2.7 (VBUS), C1.1, C2.1, DF1.2 (A), DF2.2 (A), DF3.2 (A), DF4.2 (A), J1.1 (VBUS), J2.1 (VBUS), J3.1 (VBUS), J4.1 (VBUS), J?.2 (Pin_2), R16.1, U0.3 (VI)
- net GND: now reaches U2.15 (GND), U2.23 (GND), U2.35 (GND), U2.43 (GND)
- net GND: now also U2.5 (UGND), C1.2, C15.1, C16.1, C18.2, C2.2, C5.2, C6.2, C7.2, C8.2, FB2.1, J1.4 (GND), J2.4 (GND), J3.4 (GND), J4.4 (GND), J?.8 (Pin_8), R18.2, R19.2, SW0.2 (B), U1.13 (AGND), U1.17 (AGND), U1.2 (AGND), U1.21 (AGND), U1.8 (AGND)
- net at U2.16 (XTAL2): now also C15.2, R4.2, X1.3
- net at U2.17 (XTAL1): now also C16.2, R4.1, X1.1
- net row1: now reaches U2.18 (PD0)
- net row2: now reaches U2.19 (PD1)
- net row3: now reaches U2.20 (PD2)
- net row4: now reaches U2.21 (PD3)
- net row5: now reaches U2.22 (PD5)
- net col7: now reaches U2.25 (PD4)
- net col13: now reaches U2.26 (PD6)
- net col12: now reaches U2.27 (PD7)
- net col11: now reaches U2.28 (PB4)
- net col10: now reaches U2.29 (PB5)
- net at U2.3 (D-): now also R12.1
- net col6: now reaches U2.30 (PB6)
- net col15: now reaches U2.31 (PC6)
- net at U2.33 (~HWB~/PE2): now also R19.1
- net GPIO0: now reaches U2.36 (PF7)
- net GPIO0: now also J5.21 (Pin_21), R20.1
- net GPIO1: now reaches U2.37 (PF6)
- net GPIO1: now also J5.22 (Pin_22), R21.1
- net GPIO2: now reaches U2.38 (PF5)
- net GPIO2: now also J5.23 (Pin_23), R22.1
- net GPIO3: now reaches U2.39 (PF4)
- net GPIO3: now also J5.24 (Pin_24), R23.1
- net at U2.4 (D+): now also R11.1
- net col2: now reaches U2.40 (PF1)
- net col1: now reaches U2.41 (PF0)
- net at U2.6 (UCAP): now also C18.1
- net col8: now reaches U2.9 (PB1)
- net col8: now also J?.1 (Pin_1)
- new net: R18.1, U1.11 (RREF)
- new net: C14.2, R3.1, U1.14 (X1), X2.1
- new net: C13.2, R3.2, U1.15 (X2), X2.3
- new net: R13.1, U1.37 (SPELF)
- new net: R14.1, U1.40 (PGANG/SUSPND)
- new net: R15.1, U1.41 (OVCUR#)
- new net: J1.3 (D+), R2.1
- new net: J1.2 (D-), R1.2
- new net: J2.2 (D-), R5.2
- new net: J2.3 (D+), R6.1
- new net: J3.2 (D-), R7.2
- new net: J3.3 (D+), R8.1
- new net: J4.2 (D-), R9.2
- new net: J4.3 (D+), R10.1
- new net: DF1.1 (K), R20.2
- new net: DF2.1 (K), R21.2
- new net: DF3.1 (K), R22.2
- new net: DF4.1 (K), R23.2
- new net AVCC: C5.1, C6.1, C7.1, C8.1, FB1.1, U1.1 (AVDD), U1.12 (AVDD), U1.16 (AVDD), U1.20 (AVDD), U1.7 (AVDD)
- new net DGND: C10.2, C11.2, C12.2, C13.1, C14.1, C19.2, C4.2, C9.2, FB2.2, R13.2, U0.1 (GND), U1.26 (DGND), U1.33 (DGND), U1.38 (DGND), U1.39 (TEST), U1.43 (DGND), U1.47 (DGND)
- new net DM0: R1.1, U1.3 (DM0)
- new net DM1: R11.2, U1.5 (DM1)
- new net DM2: R5.1, U1.9 (DM2)
- new net DM3: R7.1, U1.18 (DM3)
- new net DM4: R9.1, U1.22 (DM4)
- new net DP0: R2.2, U1.4 (DP0)
- new net DP1: R12.2, U1.6 (DP1)
- new net DP2: R6.2, U1.10 (DP2)
- new net DP3: R8.2, U1.19 (DP3)
- new net DP4: R10.2, U1.23 (DP4)
- new net DVCC: C10.1, C11.1, C12.1, C4.1, C9.1, FB1.2, R14.2, R15.2, R17.1, U0.2 (VO), U1.27 (DVDD), U1.34 (DVDD), U1.39 (TEST), U1.44 (DVDD)
- new net RESET1#: C19.1, R17.2, U1.28 (RESET#)
- new net lcol1: J5.6 (Pin_6)
- new net lcol10: J5.15 (Pin_15)
- new net lcol11: J5.16 (Pin_16)
- new net lcol12: J5.17 (Pin_17)
- new net lcol13: J5.18 (Pin_18)
- new net lcol14: J5.19 (Pin_19)
- new net lcol2: J5.7 (Pin_7)
- new net lcol3: J5.8 (Pin_8)
- new net lcol4: J5.9 (Pin_9)
- new net lcol5: J5.10 (Pin_10)
- new net lcol6: J5.11 (Pin_11)
- new net lcol7: J5.12 (Pin_12)
- new net lcol8: J5.13 (Pin_13)
- new net lcol9: J5.14 (Pin_14)
- new net lrow1: J5.1 (Pin_1)
- new net lrow2: J5.2 (Pin_2)
- new net lrow3: J5.3 (Pin_3)
- new net lrow4: J5.4 (Pin_4)
- new net lrow5: J5.5 (Pin_5)
- no-connect marks 0 -> 17
Other:
- moved on the sheet: U2

Commit message: complete matrix
Parts:
- gave numbers to parts that had none: 1
Changed lines of the file:
@@
 $EndComp
 $Comp
-L power:VCC #PWR?
+L power:VCC #PWR0101
 U 1 1 5BE91AC7
 P 4850 1000
-F 0 "#PWR?" H 4850 850 50  0001 C CNN
+F 0 "#PWR0101" H 4850 850 50  0001 C CNN
 F 1 "VCC" H 4867 1173 50  0000 C CNN
 F 2 "" H 4850 1000 50  0001 C CNN
@@
 $EndComp
 $Comp
-L power:VCC #PWR?
+L power:VCC #PWR0102
 U 1 1 5BE938A8
 P 700 1150
-F 0 "#PWR?" H 700 1000 50  0001 C CNN
+F 0 "#PWR0102" H 700 1000 50  0001 C CNN
 F 1 "VCC" H 717 1323 50  0000 C CNN
 F 2 "" H 700 1150 50  0001 C CNN
@@
 $EndComp
 $Comp
-L power:GND #PWR?
+L power:GND #PWR0103
 U 1 1 5BE9399E
 P 1250 1450
-F 0 "#PWR?" H 1250 1200 50  0001 C CNN
+F 0 "#PWR0103" H 1250 1200 50  0001 C CNN
 F 1 "GND" H 1255 1277 50  0000 C CNN
 F 2 "" H 1250 1450 50  0001 C CNN
@@
 $EndComp
 $Comp
-L power:GND #PWR?
+L power:GND #PWR0104
 U 1 1 5BE94BC9
 P 1000 1450
-F 0 "#PWR?" H 1000 1200 50  0001 C CNN
+F 0 "#PWR0104" H 1000 1200 50  0001 C CNN
 F 1 "GND" H 1005 1277 50  0000 C CNN
 F 2 "" H 1000 1450 50  0001 C CNN
@@
 $EndComp
 $Comp
-L power:GND #PWR?
+L power:GND #PWR0105
 U 1 1 5BE94C0B
 P 2900 1450
-F 0 "#PWR?" H 2900 1200 50  0001 C CNN
+F 0 "#PWR0105" H 2900 1200 50  0001 C CNN
 F 1 "GND" H 2905 1277 50  0000 C CNN
 F 2 "" H 2900 1450 50  0001 C CNN
@@
 $EndComp
 $Comp
-L power:GND #PWR?
+L power:GND #PWR0106
 U 1 1 5BE9DAD0
 P 5450 6150
-F 0 "#PWR?" H 5450 5900 50  0001 C CNN
+F 0 "#PWR0106" H 5450 5900 50  0001 C CNN
 F 1 "GND" H 5455 5977 50  0000 C CNN
 F 2 "" H 5450 6150 50  0001 C CNN
@@
 $EndComp
 $Comp
-L power:VCC #PWR?
+L power:VCC #PWR0107
 U 1 1 5BE9E8E4
 P 850 6700
-F 0 "#PWR?" H 850 6550 50  0001 C CNN
+F 0 "#PWR0107" H 850 6550 50  0001 C CNN
 F 1 "VCC" H 867 6873 50  0000 C CNN
 F 2 "" H 850 6700 50  0001 C CNN
@@
 $EndComp
 $Comp
-L power:VCC #PWR?
+L power:VCC #PWR0108
 U 1 1 5BE9E906
 P 2150 6700
-F 0 "#PWR?" H 2150 6550 50  0001 C CNN
+F 0 "#PWR0108" H 2150 6550 50  0001 C CNN
 F 1 "VCC" H 2167 6873 50  0000 C CNN
 F 2 "" H 2150 6700 50  0001 C CNN
@@
 $EndComp
 $Comp
-L power:VCC #PWR?
+L power:VCC #PWR0109
 U 1 1 5BE9E928
 P 3500 6700
-F 0 "#PWR?" H 3500 6550 50  0001 C CNN
+F 0 "#PWR0109" H 3500 6550 50  0001 C CNN
 F 1 "VCC" H 3517 6873 50  0000 C CNN
 F 2 "" H 3500 6700 50  0001 C CNN
@@
 $EndComp
 $Comp
-L power:GND #PWR?
+L power:GND #PWR0110
 U 1 1 5BE9EE0C
 P 3800 2350
-F 0 "#PWR?" H 3800 2100 50  0001 C CNN
+F 0 "#PWR0110" H 3800 2100 50  0001 C CNN
 F 1 "GND" H 3805 2177 50  0000 C CNN
 F 2 "" H 3800 2350 50  0001 C CNN
@@
 $EndComp
 $Comp
-L power:GND #PWR?
+L power:GND #PWR0111
 U 1 1 5BE9EE2E
 P 4500 2350
-F 0 "#PWR?" H 4500 2100 50  0001 C CNN
+F 0 "#PWR0111" H 4500 2100 50  0001 C CNN
 F 1 "GND" H 4505 2177 50  0000 C CNN
 F 2 "" H 4500 2350 50  0001 C CNN
@@
 DVCC
 $Comp
-L power:VCC #PWR?
+L power:VCC #PWR0112
 U 1 1 5BF0D43E
 P 4400 4500
-F 0 "#PWR?" H 4400 4350 50  0001 C CNN
+F 0 "#PWR0112" H 4400 4350 50  0001 C CNN
 F 1 "VCC" H 4417 4673 50  0000 C CNN
 F 2 "" H 4400 4500 50  0001 C CNN
@@
 $EndComp
 $Comp
-L power:VCC #PWR?
+L power:VCC #PWR0113
 U 1 1 5BF16B55
 P 5450 2400
-F 0 "#PWR?" H 5450 2250 50  0001 C CNN
+F 0 "#PWR0113" H 5450 2250 50  0001 C CNN
 F 1 "VCC" H 5467 2573 50  0000 C CNN
 F 2 "" H 5450 2400 50  0001 C CNN
@@
 	5450 6150 5450 6050
 $Comp
-L power:VCC #PWR?
+L power:VCC #PWR0114
 U 1 1 5BF1C053
 P 4750 3550
-F 0 "#PWR?" H 4750 3400 50  0001 C CNN
+F 0 "#PWR0114" H 4750 3400 50  0001 C CNN
 F 1 "VCC" H 4767 3723 50  0000 C CNN
 F 2 "" H 4750 3550 50  0001 C CNN
@@
 	4000 5400 4000 5500
 $Comp
-L power:GND #PWR?
+L power:GND #PWR0115
 U 1 1 5BF3F3F1
 P 4000 5800
-F 0 "#PWR?" H 4000 5550 50  0001 C CNN
+F 0 "#PWR0115" H 4000 5550 50  0001 C CNN
 F 1 "GND" H 4005 5627 50  0000 C CNN
 F 2 "" H 4000 5800 50  0001 C CNN
@@
 $EndComp
 $Comp
-L power:GND #PWR?
+L power:GND #PWR0116
 U 1 1 5BF417D5
 P 4550 4050
-F 0 "#PWR?" H 4550 3800 50  0001 C CNN
+F 0 "#PWR0116" H 4550 3800 50  0001 C CNN
 F 1 "GND" H 4555 3877 50  0000 C CNN
 F 2 "" H 4550 4050 50  0001 C CNN
@@
 $EndComp
 $Comp
-L power:GND #PWR?
+L power:GND #PWR0117
 U 1 1 5BF460BE
 P 1650 7300
-F 0 "#PWR?" H 1650 7050 50  0001 C CNN
+F 0 "#PWR0117" H 1650 7050 50  0001 C CNN
 F 1 "GND" H 1655 7127 50  0000 C CNN
 F 2 "" H 1650 7300 50  0001 C CNN
@@
 $EndComp
 $Comp
-L power:GND #PWR?
+L power:GND #PWR0118
 U 1 1 5BF46C6F
 P 2950 7300
-F 0 "#PWR?" H 2950 7050 50  0001 C CNN
+F 0 "#PWR0118" H 2950 7050 50  0001 C CNN
 F 1 "GND" H 2955 7127 50  0000 C CNN
 F 2 "" H 2950 7300 50  0001 C CNN
@@
 $EndComp
 $Comp
-L power:GND #PWR?
+L power:GND #PWR0119
 U 1 1 5BF47820
 P 4250 7300
-F 0 "#PWR?" H 4250 7050 50  0001 C CNN
+F 0 "#PWR0119" H 4250 7050 50  0001 C CNN
 F 1 "GND" H 4255 7127 50  0000 C CNN
 F 2 "" H 4250 7300 50  0001 C CNN
@@
 $EndComp
 $Comp
-L power:GND #PWR?
+L power:GND #PWR0120
 U 1 1 5BF683E6
 P 4400 5450
-F 0 "#PWR?" H 4400 5200 50  0001 C CNN
+F 0 "#PWR0120" H 4400 5200 50  0001 C CNN
 F 1 "GND" H 4405 5277 50  0000 C CNN
 F 2 "" H 4400 5450 50  0001 C CNN
@@
 	4400 4950 4400 5050
 $Comp
-L power:GND #PWR?
+L power:GND #PWR0121
 U 1 1 5BF6F7C7
 P 3500 1000
-F 0 "#PWR?" H 3500 750 50  0001 C CNN
+F 0 "#PWR0121" H 3500 750 50  0001 C CNN
 F 1 "GND" H 3505 827 50  0000 C CNN
 F 2 "" H 3500 1000 50  0001 C CNN
@@
 AVCC
 $Comp
-L power:GND #PWR?
+L power:GND #PWR0122
 U 1 1 5C063F8F
 P 8550 1150
-F 0 "#PWR?" H 8550 900 50  0001 C CNN
+F 0 "#PWR0122" H 8550 900 50  0001 C CNN
 F 1 "GND" H 8555 977 50  0000 C CNN
 F 2 "" H 8550 1150 50  0001 C CNN
@@
 lcol14
 $Comp
-L power:GND #PWR?
+L power:GND #PWR0123
 U 1 1 5C28D2BB
 P 2050 5550
-F 0 "#PWR?" H 2050 5300 50  0001 C CNN
+F 0 "#PWR0123" H 2050 5300 50  0001 C CNN
 F 1 "GND" H 2055 5377 50  0000 C CNN
 F 2 "" H 2050 5550 50  0001 C CNN
@@
 $EndComp
 $Comp
-L power:VCC #PWR?
+L power:VCC #PWR0124
 U 1 1 5C54203C
 P 10750 5050
-F 0 "#PWR?" H 10750 4900 50  0001 C CNN
+F 0 "#PWR0124" H 10750 4900 50  0001 C CNN
 F 1 "VCC" H 10767 5223 50  0000 C CNN
 F 2 "" H 10750 5050 50  0001 C CNN
@@
 $EndComp
 $Comp
-L power:GND #PWR?
+L power:GND #PWR0125
 U 1 1 5C572660
 P 6400 6350
-F 0 "#PWR?" H 6400 6100 50  0001 C CNN
+F 0 "#PWR0125" H 6400 6100 50  0001 C CNN
 F 1 "GND" H 6405 6177 50  0000 C CNN
 F 2 "" H 6400 6350 50  0001 C CNN
@@
 RESET2#
 $Comp
-L power:VCC #PWR?
+L power:VCC #PWR0126
 U 1 1 5C65890B
 P 6650 1300
-F 0 "#PWR?" H 6650 1150 50  0001 C CNN
+F 0 "#PWR0126" H 6650 1150 50  0001 C CNN
 F 1 "VCC" H 6667 1473 50  0000 C CNN
 F 2 "" H 6650 1300 50  0001 C CNN
@@
 $EndComp
 $Comp
-L power:GND #PWR?
+L power:GND #PWR0127
 U 1 1 5C6589AA
 P 6550 1900
-F 0 "#PWR?" H 6550 1650 50  0001 C CNN
+F 0 "#PWR0127" H 6550 1650 50  0001 C CNN
 F 1 "GND" H 6555 1727 50  0000 C CNN
 F 2 "" H 6550 1900 50  0001 C CNN
@@
 	6150 1800 6550 1800
 $Comp
-L Connector:Conn_01x08_Male J?
+L Connector:Conn_01x08_Male J6
 U 1 1 5C685CF0
 P 5950 1500
-F 0 "J?" H 6056 1978 50  0000 C CNN
+F 0 "J6" H 6056 1978 50  0000 C CNN
 F 1 "Conn_01x08_Male" H 6056 1887 50  0000 C CNN
 F 2 "" H 5950 1500 50  0001 C CNN

Commit message: gogogogit pull!
Parts:
- added DF1: 0603G, LED_SMD:LED_1206_3216Metric_Pad1.42x1.75mm_HandSolder, symbol Device:LED_Small
- added R20: 300, Resistor_SMD:R_0805_2012Metric_Pad1.15x1.40mm_HandSolder, symbol Device:R
- C1: footprint (none) -> Capacitor_SMD:C_1206_3216Metric_Pad1.42x1.75mm_HandSolder
- C10: renamed from C18; footprint (none) -> Capacitor_SMD:C_0805_2012Metric_Pad1.15x1.40mm_HandSolder
- C11: renamed from C5; footprint (none) -> Capacitor_SMD:C_0805_2012Metric_Pad1.15x1.40mm_HandSolder
- C12: renamed from C6; footprint (none) -> Capacitor_SMD:C_0805_2012Metric_Pad1.15x1.40mm_HandSolder
- C13: renamed from C7; footprint (none) -> Capacitor_SMD:C_0805_2012Metric_Pad1.15x1.40mm_HandSolder
- C14: renamed from C8; footprint (none) -> Capacitor_SMD:C_0805_2012Metric_Pad1.15x1.40mm_HandSolder
- C15: renamed from C9; footprint (none) -> Capacitor_SMD:C_0805_2012Metric_Pad1.15x1.40mm_HandSolder
- C16: renamed from C10; footprint (none) -> Capacitor_SMD:C_0805_2012Metric_Pad1.15x1.40mm_HandSolder
- C17: renamed from C11; footprint (none) -> Capacitor_SMD:C_0805_2012Metric_Pad1.15x1.40mm_HandSolder
- C18: renamed from C12; footprint (none) -> Capacitor_SMD:C_0805_2012Metric_Pad1.15x1.40mm_HandSolder
- C2: renamed from C19; footprint (none) -> Capacitor_SMD:C_0805_2012Metric_Pad1.15x1.40mm_HandSolder
- C3: renamed from C2; footprint (none) -> Capacitor_SMD:C_0805_2012Metric_Pad1.15x1.40mm_HandSolder
- C4: renamed from C13; footprint (none) -> Capacitor_SMD:C_0805_2012Metric_Pad1.15x1.40mm_HandSolder
- C5: renamed from C14; footprint (none) -> Capacitor_SMD:C_0805_2012Metric_Pad1.15x1.40mm_HandSolder
- C6: renamed from C3; footprint (none) -> Capacitor_SMD:C_1206_3216Metric_Pad1.42x1.75mm_HandSolder
- C7: renamed from C4; footprint (none) -> Capacitor_SMD:C_0805_2012Metric_Pad1.15x1.40mm_HandSolder
- C8: renamed from C15; footprint (none) -> Capacitor_SMD:C_0805_2012Metric_Pad1.15x1.40mm_HandSolder
- C9: renamed from C16; footprint (none) -> Capacitor_SMD:C_0805_2012Metric_Pad1.15x1.40mm_HandSolder
- DF2: renamed from DF1; footprint (none) -> LED_SMD:LED_1206_3216Metric_Pad1.42x1.75mm_HandSolder
- DF3: renamed from DF2; footprint (none) -> LED_SMD:LED_1206_3216Metric_Pad1.42x1.75mm_HandSolder
- DF4: renamed from DF3; footprint (none) -> LED_SMD:LED_1206_3216Metric_Pad1.42x1.75mm_HandSolder
- DF5: renamed from DF4; footprint (none) -> LED_SMD:LED_1206_3216Metric_Pad1.42x1.75mm_HandSolder
- FB1, FB2: footprint (none) -> Inductor_SMD:L_0805_2012Metric_Pad1.15x1.40mm_HandSolder
- J1: renamed from J2; footprint (none) -> mykeyboard:USB-A
- J2: renamed from J3; footprint (none) -> mykeyboard:USB-A
- J3: renamed from J4; footprint (none) -> mykeyboard:USB-A
- J4: renamed from J1; footprint (none) -> Connector_USB:USB_B_OST_USB-B1HSxx_Horizontal
- J5: renamed from J6; footprint (none) -> Connector_PinSocket_1.27mm:PinSocket_2x04_P1.27mm_Vertical
- J6: renamed from J5; footprint (none) -> Connector_PinSocket_1.27mm:PinSocket_2x12_P1.27mm_Vertical
- R1: renamed from R17; footprint (none) -> Resistor_SMD:R_0805_2012Metric_Pad1.15x1.40mm_HandSolder
- R10, R16, R19, R8: footprint (none) -> Resistor_SMD:R_0805_2012Metric_Pad1.15x1.40mm_HandSolder
- R11: renamed from R9; footprint (none) -> Resistor_SMD:R_0805_2012Metric_Pad1.15x1.40mm_HandSolder
- R12: renamed from R1; footprint (none) -> Resistor_SMD:R_0805_2012Metric_Pad1.15x1.40mm_HandSolder
- R13: renamed from R18; footprint (none) -> Resistor_SMD:R_0805_2012Metric_Pad1.15x1.40mm_HandSolder
- R14: renamed from R2; footprint (none) -> Resistor_SMD:R_0805_2012Metric_Pad1.15x1.40mm_HandSolder
- R15: renamed from R4; footprint (none) -> Resistor_SMD:R_0805_2012Metric_Pad1.15x1.40mm_HandSolder
- R17: renamed from R11; footprint (none) -> Resistor_SMD:R_0805_2012Metric_Pad1.15x1.40mm_HandSolder
- R18: renamed from R12; footprint (none) -> Resistor_SMD:R_0805_2012Metric_Pad1.15x1.40mm_HandSolder
- R2: renamed from R6; footprint (none) -> Resistor_SMD:R_0805_2012Metric_Pad1.15x1.40mm_HandSolder
- R21: renamed from R20; footprint (none) -> Resistor_SMD:R_0805_2012Metric_Pad1.15x1.40mm_HandSolder
- R22: renamed from R21; footprint (none) -> Resistor_SMD:R_0805_2012Metric_Pad1.15x1.40mm_HandSolder
- R23: renamed from R22; footprint (none) -> Resistor_SMD:R_0805_2012Metric_Pad1.15x1.40mm_HandSolder
- R24: renamed from R23; footprint (none) -> Resistor_SMD:R_0805_2012Metric_Pad1.15x1.40mm_HandSolder
- R3: renamed from R5; footprint (none) -> Resistor_SMD:R_0805_2012Metric_Pad1.15x1.40mm_HandSolder
- R4: renamed from R14; footprint (none) -> Resistor_SMD:R_0805_2012Metric_Pad1.15x1.40mm_HandSolder
- R5: renamed from R15; footprint (none) -> Resistor_SMD:R_0805_2012Metric_Pad1.15x1.40mm_HandSolder
- R6: renamed from R3; footprint (none) -> Resistor_SMD:R_0805_2012Metric_Pad1.15x1.40mm_HandSolder
- R7: renamed from R13; footprint (none) -> Resistor_SMD:R_0805_2012Metric_Pad1.15x1.40mm_HandSolder
- R9: renamed from R7; footprint (none) -> Resistor_SMD:R_0805_2012Metric_Pad1.15x1.40mm_HandSolder
- U1: renamed from U0; footprint (none) -> mykeyboard:TLV1117-DCY
- U2: renamed from U1; footprint (none) -> Package_QFP:LQFP-48_7x7mm_P0.5mm
- X1: renamed from X2; footprint (none) -> Crystal:Crystal_SMD_3225-4Pin_3.2x2.5mm_HandSoldering
- X2: renamed from X1; footprint (none) -> Crystal:Crystal_SMD_3225-4Pin_3.2x2.5mm_HandSoldering
- renumbered SW0 to SW1, U2 to U3
Connections:
- net DGND: now also C6.2
- net DVCC: now also C6.1
- net VCC: now also DF1.2 (A)
- net caps_led: now also R20.1
- new net: DF1.1 (K), R20.2

Commit message: junk,but still a good prove.
Parts:
- SW1: footprint (none) -> mykeyboard:SW
Changed lines of the file:
@@
 F 0 "SW1" V 4354 5348 50  0000 L CNN
 F 1 "SW_SPST" V 4445 5348 50  0000 L CNN
-F 2 "" H 4400 5250 50  0001 C CNN
+F 2 "mykeyboard:SW" H 4400 5250 50  0001 C CNN
 F 3 "" H 4400 5250 50  0001 C CNN
 	1    4400 5250
